Commit message: small refactoring for piloting integration

File: smb_description/urdf/sensor_plugins/smb_robosense.gazebo.xacro (robot description, xacro)
@@ -9,5 +9,5 @@
       <xacro:include filename="$(find robosense_description)/urdf/RS-16.urdf.xacro"/>
       <xacro:RS-16 parent="${base_link}" name="rslidar" topic="$(arg pointcloud_topic)" hz="10" samples="440" gpu="${gpu}">
-        <origin xyz="0.00445 0 ${0.298+chassisHeight/2.0}" rpy="0 0 ${M_PI/2.0}" />
+        <origin xyz="0 0 ${lidar_height_over_mount}" rpy="0 0 ${M_PI/2.0}" />
       </xacro:RS-16>
       <gazebo reference="rslidar_base_mount_joint">
@@ -41,5 +41,5 @@
         <parent link="${base_link}"/>
         <child link="rslidar"/>
-        <origin xyz="0.00445 0 ${0.298+chassisHeight/2.0+0.038}" rpy="0 0 ${M_PI/2.0}"/>
+        <origin xyz="0 0 ${lidar_height_over_mount}" rpy="0 0 ${M_PI/2.0}"/>
       </joint>
     </xacro:unless>

File: smb_description/urdf/smb.urdf.xacro (robot description, xacro)
@@ -59,11 +59,11 @@
             <joint name="${prefix}_WHEEL_JOINT">
                 <hardwareInterface>hardware_interface/VelocityJointInterface</hardwareInterface>
-                <hardwareInterface>hardware_interface/EffortJointInterface</hardwareInterface>
-                <hardwareInterface>hardware_interface/PositionJointInterface</hardwareInterface>
+             <!--    <hardwareInterface>hardware_interface/EffortJointInterface</hardwareInterface>
+                <hardwareInterface>hardware_interface/PositionJointInterface</hardwareInterface> -->
             </joint>
             <actuator name="${prefix}_WHEEL_ACTUATOR">
                 <hardwareInterface>hardware_interface/VelocityJointInterface</hardwareInterface>
-                <hardwareInterface>hardware_interface/EffortJointInterface</hardwareInterface>
-                <hardwareInterface>hardware_interface/PositionJointInterface</hardwareInterface>
+                <!-- <hardwareInterface>hardware_interface/EffortJointInterface</hardwareInterface>
+                <hardwareInterface>hardware_interface/PositionJointInterface</hardwareInterface> -->
                 <mechanicalReduction>${transmission_reduction}</mechanicalReduction>
             </actuator>
@@ -162,6 +162,6 @@
         <xacro:blackfly_cam_stereo base_link="${base_link_name}" simulation="${simulation}"/>
         <xacro:if value="${lidar}">
-            <xacro:LIDAR base_link="${base_link_name}" simulation="${simulation}"/>
             <xacro:lidar_mount base_link="${base_link_name}"/>
+            <xacro:LIDAR base_link="lidar_mount_link" simulation="${simulation}"/>
         </xacro:if>
         <xacro:if value="${tracking_camera}">

File: smb_description/urdf/smb_piloting_properties.urdf.xacro (robot description, xacro)
@@ -22,5 +22,5 @@
     <!-- Imu  Properties -->
     <xacro:property name="mount_origin_rpy"     value="0 0 0"/>
-    <xacro:property name="mount_origin_xyz"     value="0.00445 0 ${0.228+chassisHeight/2.0}"/>
-    <xacro:property name="lidar_height_over_mount" value="0.038" />
+    <xacro:property name="mount_origin_xyz"     value="0.245 0 ${0.228+chassisHeight/2.0}"/>
+    <xacro:property name="lidar_height_over_mount" value="0.14" />
 </robot>

File: smb_description/urdf/smb_properties.urdf.xacro (robot description, xacro)
@@ -1,4 +1,5 @@
 <?xml version="1.0"?>
 <robot xmlns:xacro="http://www.ros.org/wiki/xacro" name="smb">
+    <xacro:property name="base_link_name" value="base_link"/>
     <xacro:property name="chassisHeight" value="0.197"/>
     <xacro:property name="chassisLength" value="0.605"/>
@@ -17,3 +18,6 @@
     <xacro:property name="wheelHeight" value="0.08"/>
     <xacro:property name="wheelMass" value="5"/>
+    <!-- Imu  Properties -->
+    <xacro:property name="mount_origin_rpy"     value="0 0 0"/>
+    <xacro:property name="mount_origin_xyz"     value="0.00445 0 ${0.228+chassisHeight/2.0}"/>
 </robot>
