Commit message: optional changes for piloting demo

File: smb_description/urdf/sensor_plugins/smb_odometry.gazebo.xacro (robot description, xacro)
@@ -1,5 +1,5 @@
 <?xml version="1.0"?>
 <robot xmlns:xacro="http://www.ros.org/wiki/xacro" name="smb">
-<xacro:macro name="odometry_plugin" params="sensor_link topic_name odom_frame:=camera_odom_frame child_odom_frame:=camera_pose_frame publish_tf:=true rate:=20 max_linear_speed_before_settle:=0.001 max_angular_speed_before_settle:=0.001">
+<xacro:macro name="odometry_plugin" params="sensor_link topic_name odom_frame:=camera_odom_frame child_odom_frame:=camera_pose_frame publish_tf:=true rate:=20 max_linear_speed_before_settle:=0.01 max_angular_speed_before_settle:=0.1">
     <gazebo>
         <plugin name="smb_odometry_plugin" filename="libodometry_source_plugin.so">
